File: hardware/rev_a/RailLed.kicad_pcb (KiCad board)
At the start: 2 copper layers, 0 parts

Commit message: Fab out
Parts:
- added C0: CAP_0603, receiver:0603, F.Cu at (35.5, 111.5)
- added C1: CAP_0603, receiver:0603, F.Cu at (56.3, 35.4)
- added C10: CAP_0603, receiver:0603, F.Cu at (40.5, 108.0)
- added C11: CAP_0603, receiver:0603, F.Cu at (39.0, 110.0)
- added C12: CAP_0603, receiver:0603, F.Cu at (43.0, 108.0)
- added C13: CAP_0603, receiver:0603, F.Cu at (50.5, 108.0)
- added C14: CAP_0603, receiver:0603, F.Cu at (49.0, 110.0)
- added C15: CAP_0603, receiver:0603, F.Cu at (53.0, 108.0)
- added C16: CAP_0603, receiver:0603, F.Cu at (60.5, 108.0)
- added C17: CAP_0603, receiver:0603, F.Cu at (59.0, 110.0)
- added C18: CAP_0603, receiver:0603, F.Cu at (63.0, 108.0)
- added C19: CAP_0603, receiver:0603, F.Cu at (70.5, 108.0)
- added C2: CAP_0603, receiver:0603, F.Cu at (66.3, 35.4)
- added C20: CAP_0603, receiver:0603, F.Cu at (69.0, 110.0)
- added C21: CAP_0603, receiver:0603, F.Cu at (73.0, 108.0)
- added C22: CAP_0603, receiver:0603, F.Cu at (80.5, 108.0)
- added C23: CAP_0603, receiver:0603, F.Cu at (79.0, 110.0)
- added C24: CAP_0603, receiver:0603, F.Cu at (83.0, 108.0)
- added C25: CAP_0603, receiver:0603, F.Cu at (90.5, 108.0)
- added C26: CAP_0603, receiver:0603, F.Cu at (89.0, 110.0)
- added C27: CAP_0603, receiver:0603, F.Cu at (93.0, 108.0)
- added C28: CAP_0603, receiver:0603, F.Cu at (100.5, 108.0)
- added C29: CAP_0603, receiver:0603, F.Cu at (99.0, 110.0)
- added C3: CAP_0603, receiver:0603, F.Cu at (76.3, 35.4)
- added C30: CAP_0603, receiver:0603, F.Cu at (103.0, 108.0)
- added C4: CAP_0603, receiver:0603, F.Cu at (86.3, 35.4)
- added C5: CAP_0603, receiver:0603, F.Cu at (96.3, 35.4)
- added C6: CAP_0603, receiver:0603, F.Cu at (106.3, 35.4)
- added C7: CAP_0603, receiver:0603, F.Cu at (25.3, 63.7)
- added C8: CAP_0603, receiver:0603, F.Cu at (23.9, 63.7)
- added C9: CAP_0603, receiver:0603, F.Cu at (30.9, 63.7)
- added D0: 150060GS75000, RailLed:150060GS75000, F.Cu at (50.0, 105.0)
- added D1: 150060GS75000, RailLed:150060GS75000, F.Cu at (50.0, 100.0)
- added D10: 150060GS75000, RailLed:150060GS75000, F.Cu at (50.0, 55.0)
- added D100: 150060GS75000, RailLed:150060GS75000, F.Cu at (90.0, 85.0)
- added D101: 150060GS75000, RailLed:150060GS75000, F.Cu at (90.0, 80.0)
- added D102: 150060GS75000, RailLed:150060GS75000, F.Cu at (90.0, 75.0)
- added D103: 150060GS75000, RailLed:150060GS75000, F.Cu at (90.0, 70.0)
- added D104: 150060GS75000, RailLed:150060GS75000, F.Cu at (90.0, 65.0)
- added D105: 150060GS75000, RailLed:150060GS75000, F.Cu at (90.0, 60.0)
- added D106: 150060GS75000, RailLed:150060GS75000, F.Cu at (90.0, 55.0)
- added D107: 150060GS75000, RailLed:150060GS75000, F.Cu at (90.0, 50.0)
- added D108: 150060GS75000, RailLed:150060GS75000, F.Cu at (95.0, 50.0)
- added D109: 150060GS75000, RailLed:150060GS75000, F.Cu at (95.0, 55.0)
- added D11: 150060GS75000, RailLed:150060GS75000, F.Cu at (50.0, 50.0)
- added D110: 150060GS75000, RailLed:150060GS75000, F.Cu at (95.0, 60.0)
- added D111: 150060GS75000, RailLed:150060GS75000, F.Cu at (95.0, 65.0)
- added D112: 150060GS75000, RailLed:150060GS75000, F.Cu at (95.0, 70.0)
- added D113: 150060GS75000, RailLed:150060GS75000, F.Cu at (95.0, 75.0)
- added D114: 150060GS75000, RailLed:150060GS75000, F.Cu at (95.0, 80.0)
- added D115: 150060GS75000, RailLed:150060GS75000, F.Cu at (95.0, 85.0)
- added D116: 150060GS75000, RailLed:150060GS75000, F.Cu at (95.0, 90.0)
- added D117: 150060GS75000, RailLed:150060GS75000, F.Cu at (95.0, 95.0)
- added D118: 150060GS75000, RailLed:150060GS75000, F.Cu at (95.0, 100.0)
- added D119: 150060GS75000, RailLed:150060GS75000, F.Cu at (95.0, 105.0)
- added D12: 150060GS75000, RailLed:150060GS75000, F.Cu at (55.0, 50.0)
- added D120: 150060GS75000, RailLed:150060GS75000, F.Cu at (100.0, 105.0)
- added D121: 150060GS75000, RailLed:150060GS75000, F.Cu at (100.0, 100.0)
- added D122: 150060GS75000, RailLed:150060GS75000, F.Cu at (100.0, 95.0)
- added D123: 150060GS75000, RailLed:150060GS75000, F.Cu at (100.0, 90.0)
- added D124: 150060GS75000, RailLed:150060GS75000, F.Cu at (100.0, 85.0)
- added D125: 150060GS75000, RailLed:150060GS75000, F.Cu at (100.0, 80.0)
- added D126: 150060GS75000, RailLed:150060GS75000, F.Cu at (100.0, 75.0)
- added D127: 150060GS75000, RailLed:150060GS75000, F.Cu at (100.0, 70.0)
- added D128: 150060GS75000, RailLed:150060GS75000, F.Cu at (100.0, 65.0)
- added D129: 150060GS75000, RailLed:150060GS75000, F.Cu at (100.0, 60.0)
- added D13: 150060GS75000, RailLed:150060GS75000, F.Cu at (55.0, 55.0)
- added D130: 150060GS75000, RailLed:150060GS75000, F.Cu at (100.0, 55.0)
- added D131: 150060GS75000, RailLed:150060GS75000, F.Cu at (100.0, 50.0)
- added D132: 150060GS75000, RailLed:150060GS75000, F.Cu at (105.0, 50.0)
- added D133: 150060GS75000, RailLed:150060GS75000, F.Cu at (105.0, 55.0)
- added D134: 150060GS75000, RailLed:150060GS75000, F.Cu at (105.0, 60.0)
- added D135: 150060GS75000, RailLed:150060GS75000, F.Cu at (105.0, 65.0)
- added D136: 150060GS75000, RailLed:150060GS75000, F.Cu at (105.0, 70.0)
- added D137: 150060GS75000, RailLed:150060GS75000, F.Cu at (105.0, 75.0)
- added D138: 150060GS75000, RailLed:150060GS75000, F.Cu at (105.0, 80.0)
- added D139: 150060GS75000, RailLed:150060GS75000, F.Cu at (105.0, 85.0)
- added D14: 150060GS75000, RailLed:150060GS75000, F.Cu at (55.0, 60.0)
- added D140: 150060GS75000, RailLed:150060GS75000, F.Cu at (105.0, 90.0)
- added D141: 150060GS75000, RailLed:150060GS75000, F.Cu at (105.0, 95.0)
- added D142: 150060GS75000, RailLed:150060GS75000, F.Cu at (105.0, 100.0)
- added D143: 150060GS75000, RailLed:150060GS75000, F.Cu at (105.0, 105.0)
- added D15: 150060GS75000, RailLed:150060GS75000, F.Cu at (55.0, 65.0)
- added D16: 150060GS75000, RailLed:150060GS75000, F.Cu at (55.0, 70.0)
- added D17: 150060GS75000, RailLed:150060GS75000, F.Cu at (55.0, 75.0)
- added D18: 150060GS75000, RailLed:150060GS75000, F.Cu at (55.0, 80.0)
- added D19: 150060GS75000, RailLed:150060GS75000, F.Cu at (55.0, 85.0)
- added D2: 150060GS75000, RailLed:150060GS75000, F.Cu at (50.0, 95.0)
- added D20: 150060GS75000, RailLed:150060GS75000, F.Cu at (55.0, 90.0)
- added D21: 150060GS75000, RailLed:150060GS75000, F.Cu at (55.0, 95.0)
- added D22: 150060GS75000, RailLed:150060GS75000, F.Cu at (55.0, 100.0)
- added D23: 150060GS75000, RailLed:150060GS75000, F.Cu at (55.0, 105.0)
- added D24: 150060GS75000, RailLed:150060GS75000, F.Cu at (60.0, 105.0)
- added D25: 150060GS75000, RailLed:150060GS75000, F.Cu at (60.0, 100.0)
- added D26: 150060GS75000, RailLed:150060GS75000, F.Cu at (60.0, 95.0)
- added D27: 150060GS75000, RailLed:150060GS75000, F.Cu at (60.0, 90.0)
- added D28: 150060GS75000, RailLed:150060GS75000, F.Cu at (60.0, 85.0)
- added D29: 150060GS75000, RailLed:150060GS75000, F.Cu at (60.0, 80.0)
- added D3: 150060GS75000, RailLed:150060GS75000, F.Cu at (50.0, 90.0)
- added D30: 150060GS75000, RailLed:150060GS75000, F.Cu at (60.0, 75.0)
- added D31: 150060GS75000, RailLed:150060GS75000, F.Cu at (60.0, 70.0)
- added D32: 150060GS75000, RailLed:150060GS75000, F.Cu at (60.0, 65.0)
- added D33: 150060GS75000, RailLed:150060GS75000, F.Cu at (60.0, 60.0)
- added D34: 150060GS75000, RailLed:150060GS75000, F.Cu at (60.0, 55.0)
- added D35: 150060GS75000, RailLed:150060GS75000, F.Cu at (60.0, 50.0)
- added D36: 150060GS75000, RailLed:150060GS75000, F.Cu at (65.0, 50.0)
- added D37: 150060GS75000, RailLed:150060GS75000, F.Cu at (65.0, 55.0)
- added D38: 150060GS75000, RailLed:150060GS75000, F.Cu at (65.0, 60.0)
- added D39: 150060GS75000, RailLed:150060GS75000, F.Cu at (65.0, 65.0)
- added D4: 150060GS75000, RailLed:150060GS75000, F.Cu at (50.0, 85.0)
- added D40: 150060GS75000, RailLed:150060GS75000, F.Cu at (65.0, 70.0)
- added D41: 150060GS75000, RailLed:150060GS75000, F.Cu at (65.0, 75.0)
- added D42: 150060GS75000, RailLed:150060GS75000, F.Cu at (65.0, 80.0)
- added D43: 150060GS75000, RailLed:150060GS75000, F.Cu at (65.0, 85.0)
- added D44: 150060GS75000, RailLed:150060GS75000, F.Cu at (65.0, 90.0)
- added D45: 150060GS75000, RailLed:150060GS75000, F.Cu at (65.0, 95.0)
- added D46: 150060GS75000, RailLed:150060GS75000, F.Cu at (65.0, 100.0)
- added D47: 150060GS75000, RailLed:150060GS75000, F.Cu at (65.0, 105.0)
- added D48: 150060GS75000, RailLed:150060GS75000, F.Cu at (70.0, 105.0)
- added D49: 150060GS75000, RailLed:150060GS75000, F.Cu at (70.0, 100.0)
- added D5: 150060GS75000, RailLed:150060GS75000, F.Cu at (50.0, 80.0)
- added D50: 150060GS75000, RailLed:150060GS75000, F.Cu at (70.0, 95.0)
- added D51: 150060GS75000, RailLed:150060GS75000, F.Cu at (70.0, 90.0)
- added D52: 150060GS75000, RailLed:150060GS75000, F.Cu at (70.0, 85.0)
- added D53: 150060GS75000, RailLed:150060GS75000, F.Cu at (70.0, 80.0)
- added D54: 150060GS75000, RailLed:150060GS75000, F.Cu at (70.0, 75.0)
- added D55: 150060GS75000, RailLed:150060GS75000, F.Cu at (70.0, 70.0)
- added D56: 150060GS75000, RailLed:150060GS75000, F.Cu at (70.0, 65.0)
- added D57: 150060GS75000, RailLed:150060GS75000, F.Cu at (70.0, 60.0)
- added D58: 150060GS75000, RailLed:150060GS75000, F.Cu at (70.0, 55.0)
- added D59: 150060GS75000, RailLed:150060GS75000, F.Cu at (70.0, 50.0)
- added D6: 150060GS75000, RailLed:150060GS75000, F.Cu at (50.0, 75.0)
- added D60: 150060GS75000, RailLed:150060GS75000, F.Cu at (75.0, 50.0)
- added D61: 150060GS75000, RailLed:150060GS75000, F.Cu at (75.0, 55.0)
- added D62: 150060GS75000, RailLed:150060GS75000, F.Cu at (75.0, 60.0)
- added D63: 150060GS75000, RailLed:150060GS75000, F.Cu at (75.0, 65.0)
- added D64: 150060GS75000, RailLed:150060GS75000, F.Cu at (75.0, 70.0)
- added D65: 150060GS75000, RailLed:150060GS75000, F.Cu at (75.0, 75.0)
- added D66: 150060GS75000, RailLed:150060GS75000, F.Cu at (75.0, 80.0)
- added D67: 150060GS75000, RailLed:150060GS75000, F.Cu at (75.0, 85.0)
- added D68: 150060GS75000, RailLed:150060GS75000, F.Cu at (75.0, 90.0)
- added D69: 150060GS75000, RailLed:150060GS75000, F.Cu at (75.0, 95.0)
- added D7: 150060GS75000, RailLed:150060GS75000, F.Cu at (50.0, 70.0)
- added D70: 150060GS75000, RailLed:150060GS75000, F.Cu at (75.0, 100.0)
- added D71: 150060GS75000, RailLed:150060GS75000, F.Cu at (75.0, 105.0)
- added D72: 150060GS75000, RailLed:150060GS75000, F.Cu at (80.0, 105.0)
- added D73: 150060GS75000, RailLed:150060GS75000, F.Cu at (80.0, 100.0)
- added D74: 150060GS75000, RailLed:150060GS75000, F.Cu at (80.0, 95.0)
- added D75: 150060GS75000, RailLed:150060GS75000, F.Cu at (80.0, 90.0)
- added D76: 150060GS75000, RailLed:150060GS75000, F.Cu at (80.0, 85.0)
- added D77: 150060GS75000, RailLed:150060GS75000, F.Cu at (80.0, 80.0)
- added D78: 150060GS75000, RailLed:150060GS75000, F.Cu at (80.0, 75.0)
- added D79: 150060GS75000, RailLed:150060GS75000, F.Cu at (80.0, 70.0)
- added D8: 150060GS75000, RailLed:150060GS75000, F.Cu at (50.0, 65.0)
- added D80: 150060GS75000, RailLed:150060GS75000, F.Cu at (80.0, 65.0)
- added D81: 150060GS75000, RailLed:150060GS75000, F.Cu at (80.0, 60.0)
- added D82: 150060GS75000, RailLed:150060GS75000, F.Cu at (80.0, 55.0)
- added D83: 150060GS75000, RailLed:150060GS75000, F.Cu at (80.0, 50.0)
- added D84: 150060GS75000, RailLed:150060GS75000, F.Cu at (85.0, 50.0)
- added D85: 150060GS75000, RailLed:150060GS75000, F.Cu at (85.0, 55.0)
- added D86: 150060GS75000, RailLed:150060GS75000, F.Cu at (85.0, 60.0)
- added D87: 150060GS75000, RailLed:150060GS75000, F.Cu at (85.0, 65.0)
- added D88: 150060GS75000, RailLed:150060GS75000, F.Cu at (85.0, 70.0)
- added D89: 150060GS75000, RailLed:150060GS75000, F.Cu at (85.0, 75.0)
- added D9: 150060GS75000, RailLed:150060GS75000, F.Cu at (50.0, 60.0)
- added D90: 150060GS75000, RailLed:150060GS75000, F.Cu at (85.0, 80.0)
- added D91: 150060GS75000, RailLed:150060GS75000, F.Cu at (85.0, 85.0)
- added D92: 150060GS75000, RailLed:150060GS75000, F.Cu at (85.0, 90.0)
- added D93: 150060GS75000, RailLed:150060GS75000, F.Cu at (85.0, 95.0)
- added D94: 150060GS75000, RailLed:150060GS75000, F.Cu at (85.0, 100.0)
- added D95: 150060GS75000, RailLed:150060GS75000, F.Cu at (85.0, 105.0)
- added D96: 150060GS75000, RailLed:150060GS75000, F.Cu at (90.0, 105.0)
- added D97: 150060GS75000, RailLed:150060GS75000, F.Cu at (90.0, 100.0)
- added D98: 150060GS75000, RailLed:150060GS75000, F.Cu at (90.0, 95.0)
- added D99: 150060GS75000, RailLed:150060GS75000, F.Cu at (90.0, 90.0)
- added J0: XG8V-0331, RailLed:XG8V-0331, F.Cu at (25.0, 102.0)
- added J1: XG8V-0331, RailLed:XG8V-0331, F.Cu at (25.0, 120.0)
- added J2: XG8V-0331, RailLed:XG8V-0331, F.Cu at (25.0, 84.0)
- added J3: XG8V-0331, RailLed:XG8V-0331, F.Cu at (25.0, 76.4)
- added L0: CDRH6D38NP-100NC, RailLed:CDRH6D38NP-100NC, F.Cu at (39.4, 119.2)
- added L1: CDRH6D38NP-100NC, RailLed:CDRH6D38NP-100NC, F.Cu at (49.4, 119.2)
- added L2: CDRH6D38NP-100NC, RailLed:CDRH6D38NP-100NC, F.Cu at (59.4, 119.2)
- added L3: CDRH6D38NP-100NC, RailLed:CDRH6D38NP-100NC, F.Cu at (69.4, 119.2)
- added L4: CDRH6D38NP-100NC, RailLed:CDRH6D38NP-100NC, F.Cu at (79.4, 119.2)
- added L5: CDRH6D38NP-100NC, RailLed:CDRH6D38NP-100NC, F.Cu at (89.4, 119.2)
- added L6: CDRH6D38NP-100NC, RailLed:CDRH6D38NP-100NC, F.Cu at (99.4, 119.2)
- added R0: RES_0603, receiver:0603, F.Cu at (35.5, 108.5)
- added R1: RES_0603, receiver:0603, F.Cu at (35.5, 110.0)
- added R10: RES_0603, receiver:0603, F.Cu at (33.5, 76.4)
- added R11: RES_0603, receiver:0603, F.Cu at (37.1, 113.5)
- added R12: RES_0603, receiver:0603, F.Cu at (39.0, 111.5)
- added R13: RES_0603, receiver:0603, F.Cu at (44.5, 111.0)
- added R14: RES_0603, receiver:0603, F.Cu at (44.5, 114.0)
- added R15: RES_0603, receiver:0603, F.Cu at (46.7, 113.5)
- added R16: RES_0603, receiver:0603, F.Cu at (49.0, 111.5)
- added R17: RES_0603, receiver:0603, F.Cu at (54.5, 111.0)
- added R18: RES_0603, receiver:0603, F.Cu at (54.5, 114.0)
- added R19: RES_0603, receiver:0603, F.Cu at (56.7, 113.5)
- added R2: RES_0603, receiver:0603, F.Cu at (54.0, 33.9)
- added R20: RES_0603, receiver:0603, F.Cu at (59.0, 111.5)
- added R21: RES_0603, receiver:0603, F.Cu at (64.5, 111.0)
- added R22: RES_0603, receiver:0603, F.Cu at (64.5, 114.0)
- added R23: RES_0603, receiver:0603, F.Cu at (67.1, 113.5)
- added R24: RES_0603, receiver:0603, F.Cu at (69.0, 111.5)
- added R25: RES_0603, receiver:0603, F.Cu at (74.5, 111.0)
- added R26: RES_0603, receiver:0603, F.Cu at (74.5, 114.0)
- added R27: RES_0603, receiver:0603, F.Cu at (76.7, 113.5)
- added R28: RES_0603, receiver:0603, F.Cu at (79.0, 111.5)
- added R29: RES_0603, receiver:0603, F.Cu at (84.5, 111.0)
- added R3: RES_0603, receiver:0603, F.Cu at (64.0, 33.9)
- added R30: RES_0603, receiver:0603, F.Cu at (84.5, 114.0)
- added R31: RES_0603, receiver:0603, F.Cu at (86.9, 113.5)
- added R32: RES_0603, receiver:0603, F.Cu at (89.0, 111.5)
- added R33: RES_0603, receiver:0603, F.Cu at (94.5, 111.0)
- added R34: RES_0603, receiver:0603, F.Cu at (94.5, 114.0)
- added R35: RES_0603, receiver:0603, F.Cu at (96.8, 113.5)
- added R36: RES_0603, receiver:0603, F.Cu at (99.0, 111.5)
- added R37: RES_0603, receiver:0603, F.Cu at (104.5, 111.0)
- added R38: RES_0603, receiver:0603, F.Cu at (104.5, 114.0)
- added R4: RES_0603, receiver:0603, F.Cu at (74.0, 33.9)
- added R5: RES_0603, receiver:0603, F.Cu at (84.0, 33.9)
- added R6: RES_0603, receiver:0603, F.Cu at (94.0, 33.9)
- added R7: RES_0603, receiver:0603, F.Cu at (100.8, 33.8)
- added R8: RES_0603, receiver:0603, F.Cu at (29.6, 63.7)
- added R9: RES_0603, receiver:0603, F.Cu at (33.5, 73.8)
- added U0: TLC5947DAP, RailLed:TLC5947DAP, F.Cu at (48.8, 37.0)
- added U1: TLC5947DAP, RailLed:TLC5947DAP, F.Cu at (58.8, 37.0)
- added U10: LTC3440EMS#PBF, RailLed:LTC3440EMS#PBF, F.Cu at (62.6, 114.2)
- added U11: LTC3440EMS#PBF, RailLed:LTC3440EMS#PBF, F.Cu at (72.6, 114.2)
- added U12: LTC3440EMS#PBF, RailLed:LTC3440EMS#PBF, F.Cu at (82.6, 114.2)
- added U13: LTC3440EMS#PBF, RailLed:LTC3440EMS#PBF, F.Cu at (92.6, 114.2)
- added U14: LTC3440EMS#PBF, RailLed:LTC3440EMS#PBF, F.Cu at (102.6, 114.2)
- added U2: TLC5947DAP, RailLed:TLC5947DAP, F.Cu at (68.8, 37.0)
- added U3: TLC5947DAP, RailLed:TLC5947DAP, F.Cu at (78.8, 37.0)
- added U4: TLC5947DAP, RailLed:TLC5947DAP, F.Cu at (88.8, 37.0)
- added U5: TLC5947DAP, RailLed:TLC5947DAP, F.Cu at (98.8, 37.0)
- added U6: ESP32-WROOM-32D, BalanceBoard:ESP32-WROOM-32D, F.Cu at (22.9, 61.1)
- added U7: MIC5239-3.3YS, BalanceBoard:MIC5239-3.3YS, F.Cu at (43.0, 90.0)
- added U8: LTC3440EMS#PBF, RailLed:LTC3440EMS#PBF, F.Cu at (42.6, 114.2)
- added U9: LTC3440EMS#PBF, RailLed:LTC3440EMS#PBF, F.Cu at (52.6, 114.2)
Routing:
- net GND: track 0.00 -> 618.9 mm, vias 0 -> 51
- net /MODE: track 0.00 -> 317.0 mm, vias 0 -> 7
- net /~{SHDN1}: track 0.00 -> 247.4 mm, vias 0 -> 2
- net /~{SHDN2}: track 0.00 -> 239.5 mm, vias 0 -> 2
- net /~{SHDN3}: track 0.00 -> 224.9 mm, vias 0 -> 2
- net /~{SHDN4}: track 0.00 -> 211.2 mm, vias 0 -> 2
- net +3V3: track 0.00 -> 191.4 mm, vias 0 -> 23
- net /~{SHDN5}: track 0.00 -> 183.9 mm, vias 0 -> 2
- net /BANK5/VLED: track 0.00 -> 170.4 mm
- net /BANK6/VLED: track 0.00 -> 170.4 mm
- net /BANK4/VLED: track 0.00 -> 170.4 mm
- net /BANK2/VLED: track 0.00 -> 170.4 mm
- net /BANK1/VLED: track 0.00 -> 170.3 mm
- net /BANK3/VLED: track 0.00 -> 170.3 mm
- net /~{SHDN6}: track 0.00 -> 167.0 mm, vias 0 -> 2
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- added copper zone on B.Cu, net +3V3
- added copper zone on B.Cu, net +BATT
- added copper zone on B.Cu, net GND
- added copper zone on F.Cu, net GND
Other:
- board outline added: 100 x 100 mm
- board text added: "Ashley J. Robinson"
- board text added: "Jun 2024"
- board text added: "RevA"
